Commit message: 2-axis stabilization + SLAM + Nav2 + state machine

File: src/wall_e_bringup/urdf/wall_e.urdf.xacro (robot description, xacro)
@@ -2,13 +2,13 @@
 <robot name="wall_e" xmlns:xacro="http://www.ros.org/wiki/xacro">
   <!-- ── PROPERTIES ── -->
-  <xacro:property name="base_length"   value="0.216"/>  <!-- 8.5 inches -->
-  <xacro:property name="base_width"    value="0.46"/>   <!-- 46cm total -->
-  <xacro:property name="base_height"   value="0.56"/>   <!-- 56cm -->
+  <xacro:property name="base_length"   value="0.365"/>  <!-- 8.5 inches -->
+  <xacro:property name="base_width"    value="0.390"/>   <!-- 46cm total -->
+  <xacro:property name="base_height"   value="0.245"/>   <!-- 56cm -->
   <xacro:property name="track_width"   value="0.32"/>   <!-- 32cm center to center -->
   <xacro:property name="track_thick"   value="0.07"/>   <!-- 7cm track thickness -->
   <xacro:property name="wheel_radius"  value="0.05"/>   <!-- 5cm -->
-  <xacro:property name="cam_height"    value="0.20"/>   <!-- 20cm off ground -->
-  <xacro:property name="cam_forward"   value="0.147"/>  <!-- 14.7cm forward of center -->
-  <xacro:property name="pi"            value="3.14159265358979"/>
+  <xacro:property name="cam_height"    value="0.245"/>   <!-- 20cm off ground -->
+  <xacro:property name="cam_forward"   value="0.15"/>  <!-- 14.7cm forward of center -->
+  <!-- <xacro:property name="pi"            value="3.141592653  58979"/> -->
   <!-- ── BASE FOOTPRINT ── -->
   <link name="base_footprint"/>
