Commit message: Add Gazebo sim stack with RTAB-Map + Nav2 (Jazzy-compatible)
- URDF: cylinder wheels, sphere passive supports, damping, correct inertia
- Simulated RGBD camera sensor (gz-sim rgbd_camera, 2Hz)
- depthimage_to_laserscan, odom_to_tf broadcaster
- RTAB-Map with subscribe_scan=true for scan-based grid mapping
- Nav2 manually launched (no docking/route servers) — Jazzy compatible
- nav2_params.yaml: Jazzy plugin names (::), collision_monitor, behavior_server
- Hardware launch: removed hardcoded map path, Nav2 uses RTAB-Map /map
- Python nodes: fixed shebang to /usr/bin/python3 (miniconda conflict)
- World SDF: ODE physics, real_time_factor=1.0

Co-Authored-By: Claude Sonnet 4.6 <noreply@anthropic.com>

File: src/wall_e_bringup/urdf/wall_e.urdf.xacro (robot description, xacro)
@@ -5,7 +5,7 @@
   <xacro:property name="base_width"    value="0.390"/>   <!-- 46cm total -->
   <xacro:property name="base_height"   value="0.245"/>   <!-- 56cm -->
-  <xacro:property name="track_width"   value="0.32"/>   <!-- 32cm center to center -->
+  <xacro:property name="track_width"   value="0.46"/>   <!-- sim only: places wheels outside body -->
   <xacro:property name="track_thick"   value="0.07"/>   <!-- 7cm track thickness -->
-  <xacro:property name="wheel_radius"  value="0.05"/>   <!-- 5cm -->
+  <xacro:property name="wheel_radius"  value="0.08"/>   <!-- 8cm radius -->
   <xacro:property name="cam_height"    value="0.245"/>   <!-- 20cm off ground -->
   <xacro:property name="cam_forward"   value="0.15"/>  <!-- 14.7cm forward of center -->
@@ -16,5 +16,5 @@
     <parent link="base_footprint"/>
     <child  link="base_link"/>
-    <origin xyz="0 0 ${wheel_radius}" rpy="0 0 0"/>
+    <origin xyz="0 0 ${base_height/2 + wheel_radius}" rpy="0 0 0"/>
   </joint>
   <!-- ── BASE LINK ── -->
@@ -35,7 +35,7 @@
     <inertial>
       <mass value="4.0"/>
-      <inertia ixx="0.05" ixy="0" ixz="0"
-               iyy="0.05" iyz="0"
-               izz="0.08"/>
+      <inertia ixx="0.0707" ixy="0" ixz="0"
+               iyy="0.0644" iyz="0"
+               izz="0.0951"/>
     </inertial>
   </link>
@@ -43,6 +43,7 @@
   <link name="left_track">
     <visual>
+      <origin xyz="0 0 0" rpy="${pi/2} 0 0"/>
       <geometry>
-        <box size="${base_length} ${track_thick} ${wheel_radius*2}"/>
+        <cylinder radius="${wheel_radius}" length="${track_thick}"/>
       </geometry>
       <material name="black">
@@ -51,13 +52,14 @@
     </visual>
     <collision>
+      <origin xyz="0 0 0" rpy="${pi/2} 0 0"/>
       <geometry>
-        <box size="${base_length} ${track_thick} ${wheel_radius*2}"/>
+        <cylinder radius="${wheel_radius}" length="${track_thick}"/>
       </geometry>
     </collision>
     <inertial>
       <mass value="0.5"/>
-      <inertia ixx="0.001" ixy="0" ixz="0"
-               iyy="0.001" iyz="0"
-               izz="0.001"/>
+      <inertia ixx="0.001004" ixy="0" ixz="0"
+               iyy="0.001600" iyz="0"
+               izz="0.001004"/>
     </inertial>
   </link>
@@ -71,6 +73,7 @@
   <link name="right_track">
     <visual>
+      <origin xyz="0 0 0" rpy="${pi/2} 0 0"/>
       <geometry>
-        <box size="${base_length} ${track_thick} ${wheel_radius*2}"/>
+        <cylinder radius="${wheel_radius}" length="${track_thick}"/>
       </geometry>
       <material name="black">
@@ -79,13 +82,14 @@
     </visual>
     <collision>
+      <origin xyz="0 0 0" rpy="${pi/2} 0 0"/>
       <geometry>
-        <box size="${base_length} ${track_thick} ${wheel_radius*2}"/>
+        <cylinder radius="${wheel_radius}" length="${track_thick}"/>
       </geometry>
     </collision>
     <inertial>
       <mass value="0.5"/>
-      <inertia ixx="0.001" ixy="0" ixz="0"
-               iyy="0.001" iyz="0"
-               izz="0.001"/>
+      <inertia ixx="0.001004" ixy="0" ixz="0"
+               iyy="0.001600" iyz="0"
+               izz="0.001004"/>
     </inertial>
   </link>
@@ -143,3 +147,51 @@
     <origin xyz="0 0 0" rpy="0 0 0"/>
   </joint>
+  <!-- ── GAZEBO PLUGINS ── -->
+  <gazebo>
+    <plugin filename="gz-sim-diff-drive-system"
+            name="gz::sim::systems::DiffDrive">
+      <left_joint>left_track_joint</left_joint>
+      <right_joint>right_track_joint</right_joint>
+      <wheel_separation>${track_width}</wheel_separation>
+      <wheel_radius>${wheel_radius}</wheel_radius>
+      <odom_publish_frequency>30</odom_publish_frequency>
+      <topic>/cmd_vel</topic>
+      <odom_topic>/odom</odom_topic>
+      <frame_id>odom</frame_id>
+      <child_frame_id>base_footprint</child_frame_id>
+    </plugin>
+    <plugin filename="gz-sim-joint-state-publisher-system"
+            name="gz::sim::systems::JointStatePublisher">
+    </plugin>
+  </gazebo>
+  <!-- Make base_link visible in Gazebo -->
+  <gazebo reference="base_link">
+    <material>Gazebo/Grey</material>
+  </gazebo>
+  <gazebo reference="left_track">
+    <material>Gazebo/Black</material>
+  </gazebo>
+  <gazebo reference="right_track">
+    <material>Gazebo/Black</material>
+  </gazebo>
+  <gazebo reference="camera_link">
+    <material>Gazebo/Blue</material>
+    <sensor name="rgbd_camera" type="rgbd_camera">
+      <camera>
+        <horizontal_fov>1.204</horizontal_fov>
+        <image>
+          <width>640</width>
+          <height>480</height>
+        </image>
+        <clip>
+          <near>0.3</near>
+          <far>4.0</far>
+        </clip>
+      </camera>
+      <always_on>1</always_on>
+      <update_rate>2</update_rate>
+      <topic>/wall_e/camera</topic>
+      <gz_frame_id>camera_link</gz_frame_id>
+    </sensor>
+  </gazebo>
 </robot>

Commit message: Fix sim time sync, cmd_vel chain, and visual features for autonomous nav
- RTAB-Map DetectionRate 0→1Hz: prevents queue backup when processing
  exceeds camera frame interval, keeping map→odom TF fresh
- Camera 2Hz→5Hz: improves /scan update rate for Nav2 costmaps
- Nav2 transform_tolerance 1.5s: handles 1Hz TF update cadence from RTAB-Map
- controller_server cmd_vel remapped to /cmd_vel directly: fixes broken
  smoother chain where velocity commands never reached the diff drive
- Added 4 colored landmark boxes to test_room.sdf: plain white walls have
  zero visual keypoints; RTAB-Map needs edges and color contrast to build a map

Robot now drives to NavigateToPose goals autonomously in Gazebo sim.

Co-Authored-By: Claude Sonnet 4.6 <noreply@anthropic.com>

File: src/wall_e_bringup/urdf/wall_e.urdf.xacro (robot description, xacro)
@@ -34,8 +34,9 @@
     </collision>
     <inertial>
-      <mass value="4.0"/>
-      <inertia ixx="0.0707" ixy="0" ixz="0"
-               iyy="0.0644" iyz="0"
-               izz="0.0951"/>
+      <origin xyz="0 0 ${-base_height/4}" rpy="0 0 0"/>
+      <mass value="8.0"/>
+      <inertia ixx="0.1414" ixy="0" ixz="0"
+               iyy="0.1288" iyz="0"
+               izz="0.1902"/>
     </inertial>
   </link>
@@ -69,4 +70,5 @@
     <origin xyz="0 ${track_width/2} ${-base_height/2}" rpy="0 0 0"/>
     <axis xyz="0 1 0"/>
+    <dynamics damping="0.5" friction="0.5"/>
   </joint>
   <!-- ── RIGHT TRACK ── -->
@@ -99,4 +101,5 @@
     <origin xyz="0 ${-track_width/2} ${-base_height/2}" rpy="0 0 0"/>
     <axis xyz="0 1 0"/>
+    <dynamics damping="0.5" friction="0.5"/>
   </joint>
   <!-- ── D435 CAMERA ── -->
@@ -116,8 +119,8 @@
     </collision>
     <inertial>
-      <mass value="0.072"/>
-      <inertia ixx="0.0001" ixy="0" ixz="0"
-               iyy="0.0001" iyz="0"
-               izz="0.0001"/>
+      <mass value="0.001"/>
+      <inertia ixx="0.000001" ixy="0" ixz="0"
+               iyy="0.000001" iyz="0"
+               izz="0.000001"/>
     </inertial>
   </link>
@@ -171,8 +174,58 @@
   <gazebo reference="left_track">
     <material>Gazebo/Black</material>
+    <collision>
+      <surface>
+        <friction>
+          <ode><mu>1.5</mu><mu2>1.5</mu2></ode>
+        </friction>
+        <contact>
+          <ode><kp>1e6</kp><kd>100.0</kd><min_depth>0.001</min_depth></ode>
+        </contact>
+      </surface>
+    </collision>
   </gazebo>
   <gazebo reference="right_track">
     <material>Gazebo/Black</material>
-  </gazebo>
+    <collision>
+      <surface>
+        <friction>
+          <ode><mu>1.5</mu><mu2>1.5</mu2></ode>
+        </friction>
+        <contact>
+          <ode><kp>1e6</kp><kd>100.0</kd><min_depth>0.001</min_depth></ode>
+        </contact>
+      </surface>
+    </collision>
+  </gazebo>
+  <!-- ── PASSIVE SUPPORT SPHERES (pitch stability + free turning) ── -->
+  <xacro:macro name="support_wheel" params="name x_pos y_pos">
+    <link name="${name}">
+      <collision>
+        <geometry><sphere radius="${wheel_radius}"/></geometry>
+      </collision>
+      <inertial>
+        <mass value="0.01"/>
+        <inertia ixx="0.00001" ixy="0" ixz="0"
+                 iyy="0.00001" iyz="0"
+                 izz="0.00001"/>
+      </inertial>
+    </link>
+    <joint name="${name}_joint" type="fixed">
+      <parent link="base_link"/>
+      <child  link="${name}"/>
+      <origin xyz="${x_pos} ${y_pos} ${-base_height/2}" rpy="0 0 0"/>
+    </joint>
+    <gazebo reference="${name}">
+      <collision>
+        <surface>
+          <friction><ode><mu>0.01</mu><mu2>0.01</mu2></ode></friction>
+        </surface>
+      </collision>
+    </gazebo>
+  </xacro:macro>
+  <xacro:support_wheel name="left_front_support"  x_pos="${base_length/2 - wheel_radius}" y_pos="${track_width/2}"/>
+  <xacro:support_wheel name="left_rear_support"   x_pos="${-(base_length/2 - wheel_radius)}" y_pos="${track_width/2}"/>
+  <xacro:support_wheel name="right_front_support" x_pos="${base_length/2 - wheel_radius}" y_pos="${-track_width/2}"/>
+  <xacro:support_wheel name="right_rear_support"  x_pos="${-(base_length/2 - wheel_radius)}" y_pos="${-track_width/2}"/>
   <gazebo reference="camera_link">
     <material>Gazebo/Blue</material>
@@ -190,5 +243,5 @@
       </camera>
       <always_on>1</always_on>
-      <update_rate>2</update_rate>
+      <update_rate>5</update_rate>
       <topic>/wall_e/camera</topic>
       <gz_frame_id>camera_link</gz_frame_id>

Commit message: Fix Nav2 route_server lifecycle hang + end-to-end pipeline verified
Copied navigation_launch.py locally, removed route_server and
docking_server from lifecycle nodes (not needed for WALL-E nav).
Updated wall_e_isaac.launch.py to use local nav2 launch.

End-to-end verified 2026-06-24: Isaac Sim → ROS2 bridge → RTAB-Map
→ Nav2 → cmd_vel → WALL-E moving in sim. Goal accepted, recovery
behaviors active. Pipeline confirmed working.

Co-Authored-By: Claude Sonnet 4.6 <noreply@anthropic.com>

File: src/wall_e_bringup/urdf/wall_e.urdf.xacro (robot description, xacro)
@@ -44,7 +44,7 @@
   <link name="left_track">
     <visual>
-      <origin xyz="0 0 0" rpy="${pi/2} 0 0"/>
-      <geometry>
-        <cylinder radius="${wheel_radius}" length="${track_thick}"/>
+      <origin xyz="0 0 0" rpy="0 0 0"/>
+      <geometry>
+        <box size="${base_length} ${track_thick} ${wheel_radius * 2}"/>
       </geometry>
       <material name="black">
@@ -53,7 +53,7 @@
     </visual>
     <collision>
-      <origin xyz="0 0 0" rpy="${pi/2} 0 0"/>
-      <geometry>
-        <cylinder radius="${wheel_radius}" length="${track_thick}"/>
+      <origin xyz="0 0 0" rpy="0 0 0"/>
+      <geometry>
+        <box size="${base_length} ${track_thick} ${wheel_radius * 2}"/>
       </geometry>
     </collision>
@@ -75,7 +75,7 @@
   <link name="right_track">
     <visual>
-      <origin xyz="0 0 0" rpy="${pi/2} 0 0"/>
-      <geometry>
-        <cylinder radius="${wheel_radius}" length="${track_thick}"/>
+      <origin xyz="0 0 0" rpy="0 0 0"/>
+      <geometry>
+        <box size="${base_length} ${track_thick} ${wheel_radius * 2}"/>
       </geometry>
       <material name="black">
@@ -84,7 +84,7 @@
     </visual>
     <collision>
-      <origin xyz="0 0 0" rpy="${pi/2} 0 0"/>
-      <geometry>
-        <cylinder radius="${wheel_radius}" length="${track_thick}"/>
+      <origin xyz="0 0 0" rpy="0 0 0"/>
+      <geometry>
+        <box size="${base_length} ${track_thick} ${wheel_radius * 2}"/>
       </geometry>
     </collision>
